Commit message: cola

File: probot_description/urdf/probot_anno_with_gripper.xacro (robot description, xacro)
@@ -60,5 +60,5 @@
     <child link="link_1" />
     <axis xyz="0 1 0" />
-    <limit lower="-3.1416" upper="3.1416" effort="100" velocity="3" />
+    <limit lower="${-M_PI/2}" upper="${M_PI/2}" effort="100" velocity="3" />
   </joint>
   <link name="link_2">
@@ -89,5 +89,5 @@
     <child link="link_2" />
     <axis xyz="0 0 1" />
-    <limit lower="-2.0071" upper="2.0071" effort="100" velocity="3" />
+    <limit lower="${-M_PI/3}" upper="${M_PI/3}" effort="100" velocity="3" />
   </joint>
   <link name="link_3">
@@ -118,5 +118,5 @@
     <child link="link_3" />
     <axis xyz="0 0 1" />
-    <limit lower="-0.6981" upper="3.8397" effort="100" velocity="3" />
+    <limit lower="${-M_PI/6}" upper="${M_PI}" effort="100" velocity="3" />
   </joint>
   <link name="link_4">
@@ -147,5 +147,5 @@
     <child link="link_4" />
     <axis xyz="1 0 0" />
-    <limit lower="-3.1416" upper="3.1416" effort="100" velocity="3" />
+    <limit lower="${-M_PI/2}" upper="${M_PI/2}" effort="100" velocity="3" />
   </joint>
   <link name="link_5">
@@ -176,5 +176,5 @@
     <child link="link_5" />
     <axis xyz="0 0 1" />
-    <limit lower="-0.7854" upper="3.9270" effort="100" velocity="3" />
+    <limit lower="${-M_PI/6}" upper="${M_PI/2}" effort="100" velocity="3" />
   </joint>
   <link name="link_6">
@@ -205,5 +205,5 @@
     <child link="link_6" />
     <axis xyz="0 -1 0" />
-    <limit lower="-3.1416" upper="3.1416" effort="100" velocity="3" />
+    <limit lower="${-M_PI/2}" upper="${M_PI/2}" effort="100" velocity="3" />
   </joint>
   <link name="tool0"/>
